Commit message: refactor: make X3 a simulator-parity hardware platform

File: yahboomcar_description/urdf/yahboomcar_X3.urdf.xacro (robot description, xacro)
@@ -1,121 +1,67 @@
-<?xml version="1.0" encoding="utf-8"?>
-<robot name="yahboomcar" xmlns:xacro="http://wiki.ros.org/xacro">
-    <material name="Green">
-        <color rgba="0 0.7 0 1"/>
-    </material>
-    <material name="White">
-        <color rgba="0.7 0.7 0.7 1"/>
-    </material>
-    <xacro:property name="ns" value="$(arg ns)"/>
-    <link name="${ns}/base_footprint"/>
-    <link name="${ns}/imu_link"/>
-    <!-- common link-->
-    <xacro:macro name="common_link" params="name material path *origin">
-        <link name="${ns}/${name}">
-            <visual>
-                <geometry>
-                    <mesh filename="package://yahboomcar_description/meshes/${path}/${name}.STL"/>
-                </geometry>
-                <origin xyz="0 0 0" rpy="0 0 0"/>
-                <material name="${material}"/>
-            </visual>
-            <collision>
-                <geometry>
-                    <mesh filename="package://yahboomcar_description/meshes/${path}/${name}.STL"/>
-                </geometry>
-                <origin xyz="0 0 0" rpy="0 0 0"/>
-            </collision>
-            <xacro:insert_block name="origin"/>
-        </link>
-    </xacro:macro>
-    <!-- continuous joint-->
-    <xacro:macro name="continuous_joint" params="name parent child xyz rpy axis">
-        <joint name="${ns}/${name}" type="continuous">
-            <parent link="${ns}/${parent}"/>
-            <child link="${ns}/${child}"/>
-            <origin xyz="${xyz}" rpy="${rpy}"/>
-            <axis xyz="${axis}"/>
-            <limit lower="${-pi}" upper="${pi}" effort="100" velocity="1"/>
-        </joint>
-    </xacro:macro>
-    <!-- fixed joint-->
-    <xacro:macro name="fixed_joint" params="name parent child xyz rpy">
-        <joint name="${ns}/${name}" type="fixed">
-            <parent link="${ns}/${parent}"/>
-            <child link="${ns}/${child}"/>
-            <origin xyz="${xyz}" rpy="${rpy}"/>
-        </joint>
-    </xacro:macro>
-    <common_link name="base_link" material="Green" path="mecanum">
-        <inertial>
-            <origin xyz="0.00498197982182523 5.70233829969297E-05 -0.0121008098068578" rpy="0 0 0"/>
-            <mass value="0.486218814966626"/>
-            <inertia
-                    ixx="0.00196277727666921"
-                    ixy="2.50447049446755E-07"
-                    ixz="0.000140534767811098"
-                    iyy="0.00457256033711368"
-                    iyz="2.68618064993882E-07"
-                    izz="0.00493927269870476"/>
-        </inertial>
-    </common_link>
-    <fixed_joint name="base_joint" parent="base_footprint" child="base_link" xyz="0.0 0.0 0.0815" rpy="0 0 0"/>
-    <fixed_joint name="base_imu" parent="base_link" child="imu_link" xyz="-0.06 0.01 0.01" rpy="0 3.1415 1.5707"/>
-    <common_link name="front_right_wheel" material="White" path="mecanum">
-        <inertial>
-            <origin xyz="1.9051E-06 -2.3183E-07 -0.00064079" rpy="0 0 0"/>
-            <mass value="0.051532"/>
-            <inertia ixx="1.4595E-05" ixy="-4.3975E-10" ixz="4.415E-10"
-                     iyy="1.4594E-05" iyz="-1.7476E-09" izz="2.4264E-05"/>
-        </inertial>
-    </common_link>
-    <continuous_joint name="front_right_joint" parent="base_link" child="front_right_wheel"
-                      xyz="0.08 -0.0845 -0.0389" rpy="-${pi/2} 0 ${pi}" axis="0 0 1"/>
-    <common_link name="front_left_wheel" material="White" path="mecanum">
-        <inertial>
-            <origin xyz="2.3728E-06 -9.4228E-07 0.00064068" rpy="0 0 0"/>
-            <mass value="0.051543"/>
-            <inertia ixx="1.4597E-05" ixy="-4.7945E-10" ixz="-2.4786E-10"
-                     iyy="1.4598E-05" iyz="1.7972E-09" izz="2.4267E-05"/>
-        </inertial>
-    </common_link>
-    <continuous_joint name="front_left_joint" parent="base_link" child="front_left_wheel"
-                      xyz="0.08 0.084492 -0.0389" rpy="${pi/2} 0 0" axis="0 0 1"/>
-    <common_link name="back_right_wheel" material="White" path="mecanum">
-        <inertial>
-            <origin xyz="-1.75924169923403E-06 1.28388821071107E-06 -0.000590549296238266" rpy="0 0 0"/>
-            <mass value="0.051540174053366"/>
-            <inertia ixx="1.45974152250002E-05" ixy="1.94850559178397E-10" ixz="-1.61846387282284E-09"
-                     iyy="1.4596501955693E-05" iyz="-6.27904057423818E-10" izz="2.42663091380451E-05"/>
-        </inertial>
-    </common_link>
-    <continuous_joint name="back_right_joint" parent="base_link" child="back_right_wheel"
-                      xyz="-0.08 -0.0845 -0.03946" rpy="-${pi/2} 0 ${pi}" axis="0 0 1"/>
-    <common_link name="back_left_wheel" material="White" path="mecanum">
-        <inertial>
-            <origin xyz="-4.01213085227115E-07 2.04910264598596E-06 0.000590775697051377" rpy="0 0 0"/>
-            <mass value="0.0515309299357028"/>
-            <inertia ixx="1.45942986129926E-05" ixy="-3.19787215398093E-10" ixz="1.74943062058915E-09"
-                     iyy="1.45948727598913E-05" iyz="1.61769812110049E-10" izz="2.4263683888153E-05"/>
-        </inertial>
-    </common_link>
-    <continuous_joint name="back_left_joint" parent="base_link" child="back_left_wheel"
-                      xyz="-0.08 0.084492 -0.03954" rpy="${pi/2} 0 0" axis="0 0 1"/>
-    <common_link name="laser_link" material="White" path="sensor">
-        <inertial>
-            <origin xyz="-0.0176558922685589 0.000671805271544437 0.0219302095894866" rpy="0 0 0"/>
-            <mass value="0.0483909504209895"/>
-            <inertia ixx="1.58456966399128E-05" ixy="-4.23913983850005E-07" ixz="-2.09597897904374E-07"
-                     iyy="3.89262522903605E-05" iyz="3.24809725932687E-07" izz="4.86230801106223E-05"/>
-        </inertial>
-    </common_link>
-    <fixed_joint name="laser_joint" parent="base_link" child="laser_link" xyz="0.0435 5.25826986680105E-05 0.11" rpy="0 0 0"/>
-    <common_link name="camera_link" material="White" path="sensor">
-        <inertial>
-            <origin xyz="0 0 0" rpy="0 0 0"/>
-            <mass value="0"/>
-            <inertia ixx="0" ixy="0" ixz="0" iyy="0" iyz="0" izz="0"/>
-        </inertial>
-    </common_link>
-    <fixed_joint name="camera_joint" parent="base_link" child="camera_link" xyz="0.057105 1.7948E-05 0.03755" rpy="0 0 0"/>
+<?xml version="1.0"?>
+<robot name="rosmaster_x3" xmlns:xacro="http://wiki.ros.org/xacro">
+  <!--
+    Canonical physical X3 description.
+    Frame and wheel-joint names intentionally match the simulator. This model
+    owns rigid platform transforms through cam_1_link. The Orbbec driver owns
+    calibrated camera-internal frames below cam_1_link.
+  -->
+  <xacro:arg name="prefix" default=""/>
+  <xacro:property name="prefix" value="$(arg prefix)"/>
+  <material name="platform_green"><color rgba="0.0 0.7 0.0 1.0"/></material>
+  <material name="wheel_grey"><color rgba="0.25 0.25 0.25 1.0"/></material>
+  <material name="sensor_grey"><color rgba="0.65 0.65 0.65 1.0"/></material>
+  <xacro:macro name="mesh_link" params="name mesh material mass:=0.01">
+    <link name="${prefix}${name}">
+      <visual>
+        <geometry><mesh filename="package://yahboomcar_description/meshes/${mesh}"/></geometry>
+        <material name="${material}"/>
+      </visual>
+      <collision>
+        <geometry><mesh filename="package://yahboomcar_description/meshes/${mesh}"/></geometry>
+      </collision>
+      <inertial>
+        <mass value="${mass}"/>
+        <inertia ixx="0.00001" ixy="0" ixz="0" iyy="0.00001" iyz="0" izz="0.00001"/>
+      </inertial>
+    </link>
+  </xacro:macro>
+  <xacro:macro name="fixed_joint" params="name parent child xyz rpy">
+    <joint name="${prefix}${name}" type="fixed">
+      <parent link="${prefix}${parent}"/>
+      <child link="${prefix}${child}"/>
+      <origin xyz="${xyz}" rpy="${rpy}"/>
+    </joint>
+  </xacro:macro>
+  <xacro:macro name="wheel" params="position side xyz rpy mesh">
+    <xacro:mesh_link name="${position}_${side}_wheel" mesh="${mesh}" material="wheel_grey" mass="0.0515"/>
+    <joint name="${prefix}${position}_${side}_wheel_joint" type="continuous">
+      <parent link="${prefix}base_link"/>
+      <child link="${prefix}${position}_${side}_wheel"/>
+      <origin xyz="${xyz}" rpy="${rpy}"/>
+      <axis xyz="0 0 1"/>
+      <limit effort="100" velocity="20"/>
+    </joint>
+  </xacro:macro>
+  <link name="${prefix}base_footprint"/>
+  <xacro:mesh_link name="base_link" mesh="base_link_X3.STL" material="platform_green" mass="0.486"/>
+  <xacro:fixed_joint name="base_joint" parent="base_footprint" child="base_link"
+                     xyz="0 0 0.0815" rpy="0 0 0"/>
+  <xacro:wheel position="front" side="left" xyz="0.08 0.084492 -0.0389"
+               rpy="${pi/2} 0 0" mesh="front_left_wheel_X3.STL"/>
+  <xacro:wheel position="front" side="right" xyz="0.08 -0.0845 -0.0389"
+               rpy="-${pi/2} 0 ${pi}" mesh="front_right_wheel_X3.STL"/>
+  <xacro:wheel position="back" side="left" xyz="-0.08 0.084492 -0.03954"
+               rpy="${pi/2} 0 0" mesh="back_left_wheel_X3.STL"/>
+  <xacro:wheel position="back" side="right" xyz="-0.08 -0.0845 -0.03946"
+               rpy="-${pi/2} 0 ${pi}" mesh="back_right_wheel_X3.STL"/>
+  <link name="${prefix}imu_link"/>
+  <xacro:fixed_joint name="imu_joint" parent="base_link" child="imu_link"
+                     xyz="-0.06 0.01 0.01" rpy="0 ${pi} ${pi/2}"/>
+  <xacro:mesh_link name="laser_link" mesh="laser_link.STL" material="sensor_grey" mass="0.048"/>
+  <xacro:fixed_joint name="laser_joint" parent="base_link" child="laser_link"
+                     xyz="0.0435 0.0000526 0.11" rpy="0 0 0"/>
+  <xacro:mesh_link name="cam_1_link" mesh="camera_link.STL" material="sensor_grey" mass="0.01"/>
+  <xacro:fixed_joint name="camera_mount_joint" parent="base_link" child="cam_1_link"
+                     xyz="0.057105 0.000017948 0.03755" rpy="0 0 0"/>
 </robot>

Commit message: feat: use the simulator's textured CAD meshes for RViz visuals
RViz showed a plain grey model built from the legacy flat-shaded STL
set. yahboom_rosmaster generates a textured OBJ/MTL CAD-visual mesh
set from the same source geometry (verified: every retained STL here
is byte-identical to its counterpart in that repo's legacy visual
set) and uses it for its own RViz/Gazebo rendering. Point the <visual>
mesh at that set so both platforms render the same model; <collision>
keeps the original STL, unaffected.

Copied as-is from yahboom_rosmaster (BSD-3-Clause); documented in
Provenance and licensing. Verified with `xacro` that every link
resolves to the new mesh and every collision geometry is untouched.

File: yahboomcar_description/urdf/yahboomcar_X3.urdf.xacro (robot description, xacro)
@@ -12,8 +12,9 @@
   <material name="wheel_grey"><color rgba="0.25 0.25 0.25 1.0"/></material>
   <material name="sensor_grey"><color rgba="0.65 0.65 0.65 1.0"/></material>
-  <xacro:macro name="mesh_link" params="name mesh material mass:=0.01">
+  <xacro:macro name="mesh_link" params="name mesh material mass:=0.01 visual_mesh:=''">
+    <xacro:property name="effective_visual_mesh" value="${visual_mesh if visual_mesh else mesh}"/>
     <link name="${prefix}${name}">
       <visual>
-        <geometry><mesh filename="package://yahboomcar_description/meshes/${mesh}"/></geometry>
+        <geometry><mesh filename="package://yahboomcar_description/meshes/${effective_visual_mesh}"/></geometry>
         <material name="${material}"/>
       </visual>
@@ -34,6 +35,6 @@
     </joint>
   </xacro:macro>
-  <xacro:macro name="wheel" params="position side xyz rpy mesh">
-    <xacro:mesh_link name="${position}_${side}_wheel" mesh="${mesh}" material="wheel_grey" mass="0.0515"/>
+  <xacro:macro name="wheel" params="position side xyz rpy mesh visual_mesh:=''">
+    <xacro:mesh_link name="${position}_${side}_wheel" mesh="${mesh}" material="wheel_grey" mass="0.0515" visual_mesh="${visual_mesh}"/>
     <joint name="${prefix}${position}_${side}_wheel_joint" type="continuous">
       <parent link="${prefix}base_link"/>
@@ -45,22 +46,29 @@
   </xacro:macro>
   <link name="${prefix}base_footprint"/>
-  <xacro:mesh_link name="base_link" mesh="base_link_X3.STL" material="platform_green" mass="0.486"/>
+  <xacro:mesh_link name="base_link" mesh="base_link_X3.STL" material="platform_green" mass="0.486"
+                   visual_mesh="cad_visual/rosmaster_base.obj"/>
   <xacro:fixed_joint name="base_joint" parent="base_footprint" child="base_link"
                      xyz="0 0 0.0815" rpy="0 0 0"/>
   <xacro:wheel position="front" side="left" xyz="0.08 0.084492 -0.0389"
-               rpy="${pi/2} 0 0" mesh="front_left_wheel_X3.STL"/>
+               rpy="${pi/2} 0 0" mesh="front_left_wheel_X3.STL"
+               visual_mesh="cad_visual/front_left_wheel.obj"/>
   <xacro:wheel position="front" side="right" xyz="0.08 -0.0845 -0.0389"
-               rpy="-${pi/2} 0 ${pi}" mesh="front_right_wheel_X3.STL"/>
+               rpy="-${pi/2} 0 ${pi}" mesh="front_right_wheel_X3.STL"
+               visual_mesh="cad_visual/front_right_wheel.obj"/>
   <xacro:wheel position="back" side="left" xyz="-0.08 0.084492 -0.03954"
-               rpy="${pi/2} 0 0" mesh="back_left_wheel_X3.STL"/>
+               rpy="${pi/2} 0 0" mesh="back_left_wheel_X3.STL"
+               visual_mesh="cad_visual/back_left_wheel.obj"/>
   <xacro:wheel position="back" side="right" xyz="-0.08 -0.0845 -0.03946"
-               rpy="-${pi/2} 0 ${pi}" mesh="back_right_wheel_X3.STL"/>
+               rpy="-${pi/2} 0 ${pi}" mesh="back_right_wheel_X3.STL"
+               visual_mesh="cad_visual/back_right_wheel.obj"/>
   <link name="${prefix}imu_link"/>
   <xacro:fixed_joint name="imu_joint" parent="base_link" child="imu_link"
                      xyz="-0.06 0.01 0.01" rpy="0 ${pi} ${pi/2}"/>
-  <xacro:mesh_link name="laser_link" mesh="laser_link.STL" material="sensor_grey" mass="0.048"/>
+  <xacro:mesh_link name="laser_link" mesh="laser_link.STL" material="sensor_grey" mass="0.048"
+                   visual_mesh="cad_visual/lidar.obj"/>
   <xacro:fixed_joint name="laser_joint" parent="base_link" child="laser_link"
                      xyz="0.0435 0.0000526 0.11" rpy="0 0 ${pi}"/>
-  <xacro:mesh_link name="cam_1_link" mesh="camera_link.STL" material="sensor_grey" mass="0.01"/>
+  <xacro:mesh_link name="cam_1_link" mesh="camera_link.STL" material="sensor_grey" mass="0.01"
+                   visual_mesh="cad_visual/camera.obj"/>
   <xacro:fixed_joint name="camera_mount_joint" parent="base_link" child="cam_1_link"
                      xyz="0.057105 0.000017948 0.03755" rpy="0 0 0"/>

Commit message: fix: rotate wheel visual meshes to match the joint spin axis
The cad_visual wheel OBJs are authored against yahboom_rosmaster's wheel
frame, where the spin axis is Y (`<axis xyz="0 1 0"/>`). This repo's wheel
links spin about Z, so dropping the meshes in without a compensating
rotation renders all four wheels 90 degrees out: they stand in the wrong
plane and rotate about their own face instead of rolling.

Add a `visual_rpy` parameter to `mesh_link`/`wheel` and pass each wheel the
inverse of its own joint rpy, which maps the mesh spin axis back onto the
link's `<axis>`. Verified in RViz against a live robot_state_publisher: the
wheels now roll correctly under the joint sliders, and the rotated OBJ
bounding boxes match the collision STLs to within 0.2 mm on every axis.

Collision geometry and every joint origin are untouched, so the TF tree is
unchanged; this only affects what a viewer draws.

File: yahboomcar_description/urdf/yahboomcar_X3.urdf.xacro (robot description, xacro)
@@ -12,8 +12,9 @@
   <material name="wheel_grey"><color rgba="0.25 0.25 0.25 1.0"/></material>
   <material name="sensor_grey"><color rgba="0.65 0.65 0.65 1.0"/></material>
-  <xacro:macro name="mesh_link" params="name mesh material mass:=0.01 visual_mesh:=''">
+  <xacro:macro name="mesh_link" params="name mesh material mass:=0.01 visual_mesh:='' visual_rpy:='0 0 0'">
     <xacro:property name="effective_visual_mesh" value="${visual_mesh if visual_mesh else mesh}"/>
     <link name="${prefix}${name}">
       <visual>
+        <origin xyz="0 0 0" rpy="${visual_rpy}"/>
         <geometry><mesh filename="package://yahboomcar_description/meshes/${effective_visual_mesh}"/></geometry>
         <material name="${material}"/>
@@ -35,6 +36,6 @@
     </joint>
   </xacro:macro>
-  <xacro:macro name="wheel" params="position side xyz rpy mesh visual_mesh:=''">
-    <xacro:mesh_link name="${position}_${side}_wheel" mesh="${mesh}" material="wheel_grey" mass="0.0515" visual_mesh="${visual_mesh}"/>
+  <xacro:macro name="wheel" params="position side xyz rpy mesh visual_mesh:='' visual_rpy:='0 0 0'">
+    <xacro:mesh_link name="${position}_${side}_wheel" mesh="${mesh}" material="wheel_grey" mass="0.0515" visual_mesh="${visual_mesh}" visual_rpy="${visual_rpy}"/>
     <joint name="${prefix}${position}_${side}_wheel_joint" type="continuous">
       <parent link="${prefix}base_link"/>
@@ -52,14 +53,14 @@
   <xacro:wheel position="front" side="left" xyz="0.08 0.084492 -0.0389"
                rpy="${pi/2} 0 0" mesh="front_left_wheel_X3.STL"
-               visual_mesh="cad_visual/front_left_wheel.obj"/>
+               visual_mesh="cad_visual/front_left_wheel.obj" visual_rpy="${-pi/2} 0 0"/>
   <xacro:wheel position="front" side="right" xyz="0.08 -0.0845 -0.0389"
                rpy="-${pi/2} 0 ${pi}" mesh="front_right_wheel_X3.STL"
-               visual_mesh="cad_visual/front_right_wheel.obj"/>
+               visual_mesh="cad_visual/front_right_wheel.obj" visual_rpy="${-pi/2} 0 ${-pi}"/>
   <xacro:wheel position="back" side="left" xyz="-0.08 0.084492 -0.03954"
                rpy="${pi/2} 0 0" mesh="back_left_wheel_X3.STL"
-               visual_mesh="cad_visual/back_left_wheel.obj"/>
+               visual_mesh="cad_visual/back_left_wheel.obj" visual_rpy="${-pi/2} 0 0"/>
   <xacro:wheel position="back" side="right" xyz="-0.08 -0.0845 -0.03946"
                rpy="-${pi/2} 0 ${pi}" mesh="back_right_wheel_X3.STL"
-               visual_mesh="cad_visual/back_right_wheel.obj"/>
+               visual_mesh="cad_visual/back_right_wheel.obj" visual_rpy="${-pi/2} 0 ${-pi}"/>
   <link name="${prefix}imu_link"/>
   <xacro:fixed_joint name="imu_joint" parent="base_link" child="imu_link"

Commit message: fix(description): use accurate CAD collision and derive footprint offset from wheel radius
base_link's <collision> pointed at the legacy Yahboom base_link_X3.STL,
which includes a tablet mount and antennas x3-c does not have; <visual>
already used the accurate CAD mesh since #26. Point <collision> at the
same CAD mesh so they can't diverge again.

base_joint's z (0.0815) was an independent magic number with no tie to
wheel radius, leaving the wheel bottom floating ~10mm above the
footprint ground plane. Derive it from a named wheel_radius (0.0325m,
Yahboom's 65mm-diameter spec, matching the simulator) plus the measured
front-wheel mounting drop, so the contact plane can't drift again.
Also correct the odometry wheel_radius default/param (0.033 -> 0.0325)
to the same value, since it was a third, disagreeing number that
directly affects distance-scale accuracy.

Fixes #28
Fixes #29

File: yahboomcar_description/urdf/yahboomcar_X3.urdf.xacro (robot description, xacro)
@@ -46,9 +46,12 @@
     </joint>
   </xacro:macro>
+  <!-- 65 mm wheel diameter per Yahboom ROSMASTER X3 spec; matches the simulator. -->
+  <xacro:property name="wheel_radius" value="0.0325"/>
+  <!-- base_link sits this far above the front wheel axle; measured on x3-c. -->
+  <xacro:property name="front_wheel_drop" value="0.0389"/>
   <link name="${prefix}base_footprint"/>
-  <xacro:mesh_link name="base_link" mesh="base_link_X3.STL" material="platform_green" mass="0.486"
-                   visual_mesh="cad_visual/rosmaster_base.obj"/>
+  <xacro:mesh_link name="base_link" mesh="cad_visual/rosmaster_base.obj" material="platform_green" mass="0.486"/>
   <xacro:fixed_joint name="base_joint" parent="base_footprint" child="base_link"
-                     xyz="0 0 0.0815" rpy="0 0 0"/>
+                     xyz="0 0 ${front_wheel_drop + wheel_radius}" rpy="0 0 0"/>
   <xacro:wheel position="front" side="left" xyz="0.08 0.084492 -0.0389"
                rpy="${pi/2} 0 0" mesh="front_left_wheel_X3.STL"
